Commit message: used vs code with visualizer and got the model looking really good.

File: modelv3/open_rover.urdf (robot description, URDF)
Before this commit: robot open_rover, 3 links, 2 joints
Links:
- added link back_left_wheel_link, mass 2.0; collision cylinder length=0.11 radius=0.15; visual cylinder length=0.05 radius=0.008
- added link back_right_wheel_link, mass 2.0; collision cylinder length=0.11 radius=0.15; visual cylinder length=0.05 radius=0.008
- added link front_left_wheel_link, mass 2.0; collision cylinder length=0.11 radius=0.15; visual cylinder length=0.05 radius=0.008
- added link front_right_wheel_link, mass 2.0; collision cylinder length=0.11 radius=0.15; visual cylinder length=0.05 radius=0.008
Joints:
- added joint back_left_wheel_joint: type revolute, parent main_frame, child back_left_wheel_link, origin xyz=-0.36075 0.39925 -0.45275 rpy=0 0 0, axis 0 1 0, limit effort=100.0 velocity=10.0
- added joint back_right_wheel_joint: type revolute, parent main_frame, child back_right_wheel_link, origin xyz=-0.36075 -0.39925 -0.45275 rpy=0 0 0, axis 0 1 0, limit effort=100.0 velocity=10.0
- added joint front_left_wheel_joint: type revolute, parent front_rocker_link, child front_left_wheel_link, origin xyz=0.0385 0.39925 -0.45275 rpy=0 0 0, axis 0 1 0, limit effort=100.0 velocity=10.0
- added joint front_right_wheel_joint: type revolute, parent front_rocker_link, child front_right_wheel_link, origin xyz=0.0385 -0.39925 -0.45275 rpy=0 0 0, axis 0 1 0, limit effort=100.0 velocity=10.0
- joint front_rocker_joint: origin xyz=0.39925 0 0 rpy=0 0 0 -> xyz=0.36075 0 0 rpy=0 0 0
