Commit message: Update URDF to match physical design

File: src/open_rover_model/urdf/open_rover.urdf (robot description, URDF)
Before this commit: robot open_rover, 11 links, 10 joints
Links:
- removed link left_front_leg
- removed link left_front_wheel
- removed link left_rear_leg
- removed link left_rear_wheel
- removed link main_frame
- removed link pivot_frame
- removed link right_front_leg
- removed link right_front_wheel
- removed link right_rear_leg
- removed link right_rear_wheel
- added link main_frame_base, mass 1.8; collision box size=0.76 0.04 0.04; visual box size=0.76 0.04 0.04
- added link main_frame_end1, mass 1.8; collision box size=0.04 0.75 0.04; visual box size=0.04 0.75 0.04
- added link main_frame_end2, mass 1.8; collision box size=0.04 0.75 0.04; visual box size=0.04 0.75 0.04
- added link main_frame_leg1, mass 1.2; collision box size=0.04 0.04 0.5; visual box size=0.04 0.04 0.5
- added link main_frame_leg2, mass 1.2; collision box size=0.04 0.04 0.5; visual box size=0.04 0.04 0.5
- added link main_frame_side1, mass 1.8; collision box size=0.76 0.04 0.04; visual box size=0.76 0.04 0.04
- added link pivot_frame_base, mass 1.8; collision box size=0.75 0.04 0.04; visual box size=0.75 0.04 0.04
- added link pivot_frame_leg1, mass 1.2; collision box size=0.04 0.04 0.5; visual box size=0.04 0.04 0.5
- added link pivot_frame_leg2, mass 1.2; collision box size=0.04 0.04 0.5; visual box size=0.04 0.04 0.5
- added link sheet_metal_box, mass 11.3; collision box size=0.76 0.75 0.1; visual box size=0.76 0.75 0.1
Joints:
- removed joint left_front_leg_to_wheel
- removed joint left_rear_leg_to_wheel
- removed joint main_to_left_rear_leg
- removed joint main_to_pivot_frame
- removed joint main_to_right_rear_leg
- removed joint pivot_to_left_front_leg
- removed joint pivot_to_right_front_leg
- removed joint right_front_leg_to_wheel
- removed joint right_rear_leg_to_wheel
- added joint main_frame_end1_joint: type fixed, parent main_frame_base, child main_frame_end1, origin xyz=0.36 0.375 0 rpy=0 0 0
- added joint main_frame_end2_joint: type fixed, parent main_frame_base, child main_frame_end2, origin xyz=-0.36 0.375 0 rpy=0 0 0
- added joint main_frame_leg1_joint: type fixed, parent main_frame_base, child main_frame_leg1, origin xyz=0.36 0.73 0.23 rpy=0 0 0
- added joint main_frame_leg2_joint: type fixed, parent main_frame_base, child main_frame_leg2, origin xyz=-0.36 0.73 0.23 rpy=0 0 0
- added joint main_frame_side1_joint: type fixed, parent main_frame_base, child main_frame_side1, origin xyz=0 0.75 0 rpy=0 0 0
- added joint pivot_frame_leg1_joint: type fixed, parent pivot_frame_base, child pivot_frame_leg1, origin xyz=0.355 0 -0.23 rpy=0 0 0
- added joint pivot_frame_leg2_joint: type fixed, parent pivot_frame_base, child pivot_frame_leg2, origin xyz=-0.355 0 -0.23 rpy=0 0 0
- added joint pivot_joint: type revolute, parent main_frame_base, child pivot_frame_base, origin xyz=-0.38 0 0 rpy=0 0 0, axis 0 1 0, limit lower=-0.785 upper=0.785 effort=100 velocity=1.0
- added joint sheet_metal_box_joint: type fixed, parent main_frame_base, child sheet_metal_box, origin xyz=0 0.375 -0.05 rpy=0 0 0
- joint dummy_to_main_frame: child main_frame -> main_frame_base

Commit message: I'll fix the material definitions and adjust the component positions.

File: src/open_rover_model/urdf/open_rover.urdf (robot description, URDF)
Before this commit: robot open_rover, 11 links, 10 joints
Joints:
- joint main_frame_leg1_joint: origin xyz=0.36 0.73 0.23 rpy=0 0 0 -> xyz=0.36 0.73 -0.23 rpy=0 0 0
- joint main_frame_leg2_joint: origin xyz=-0.36 0.73 0.23 rpy=0 0 0 -> xyz=-0.36 0.73 -0.23 rpy=0 0 0
- joint sheet_metal_box_joint: origin xyz=0 0.375 -0.05 rpy=0 0 0 -> xyz=0 0.355 -0.05 rpy=0 0 0

Commit message: removed the other models and moved model three into the src/urdf dir.

File: src/open_rover_model/urdf/open_rover.urdf (robot description, URDF)
Before this commit: robot open_rover, 11 links, 10 joints
Links:
- removed link dummy_root
- removed link left_front_leg
- removed link left_front_wheel
- removed link left_rear_leg
- removed link left_rear_wheel
- removed link pivot_frame
- removed link right_front_leg
- removed link right_front_wheel
- removed link right_rear_leg
- removed link right_rear_wheel
- added link back_left_wheel_link, mass 2.0; collision cylinder length=0.11 radius=0.15; visual cylinder length=0.05 radius=0.008
- added link back_right_wheel_link, mass 2.0; collision cylinder length=0.11 radius=0.15; visual cylinder length=0.05 radius=0.008
- added link base_link
- added link front_left_wheel_link, mass 2.0; collision cylinder length=0.11 radius=0.15; visual cylinder length=0.05 radius=0.008
- added link front_right_wheel_link, mass 2.0; collision cylinder length=0.11 radius=0.15; visual cylinder length=0.05 radius=0.008
- added link front_rocker_link, mass 5.0; collision box size=0.0385 0.0385 0.500; collision box size=0.0385 0.0385 0.500
- link main_frame: mass 34.1 -> 15.0; geometry collision box size=0.002 0.760 0.100; collision box size=0.002 0.760 0.100
Joints:
- removed joint dummy_to_main_frame
- removed joint left_front_leg_to_wheel
- removed joint left_rear_leg_to_wheel
- removed joint main_to_left_rear_leg
- removed joint main_to_pivot_frame
- removed joint main_to_right_rear_leg
- removed joint pivot_to_left_front_leg
- removed joint pivot_to_right_front_leg
- removed joint right_front_leg_to_wheel
- removed joint right_rear_leg_to_wheel
- added joint back_left_wheel_joint: type revolute, parent main_frame, child back_left_wheel_link, origin xyz=-0.36075 0.39925 -0.45275 rpy=0 0 0, axis 0 1 0, limit effort=100.0 velocity=10.0
- added joint back_right_wheel_joint: type revolute, parent main_frame, child back_right_wheel_link, origin xyz=-0.36075 -0.39925 -0.45275 rpy=0 0 0, axis 0 1 0, limit effort=100.0 velocity=10.0
- added joint front_left_wheel_joint: type revolute, parent front_rocker_link, child front_left_wheel_link, origin xyz=0.0385 0.39925 -0.45275 rpy=0 0 0, axis 0 1 0, limit effort=100.0 velocity=10.0
- added joint front_right_wheel_joint: type revolute, parent front_rocker_link, child front_right_wheel_link, origin xyz=0.0385 -0.39925 -0.45275 rpy=0 0 0, axis 0 1 0, limit effort=100.0 velocity=10.0
- added joint front_rocker_joint: type revolute, parent base_link, child front_rocker_link, origin xyz=0.36075 0 0 rpy=0 0 0, axis 1 0 0, limit lower=-0.5236 upper=0.5236 effort=100.0 velocity=1.0
- added joint main_frame_joint: type fixed, parent base_link, child main_frame, origin xyz=0 0 0 rpy=0 0 0
